File: PatchLogic.kicad_sch (KiCad schematic)
At the start: 0 parts

Commit message: Adicionando novos datasheets e comecando power
Other:
- title: ECP5 85F Platonic Board -> PatchLogic 85 FPGA Board
Changed lines of the file:
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@@
 	(paper "A4")
 	(title_block
-		(title "ECP5 85F Platonic Board")
-		(date "2025-01-05")
+		(title "PatchLogic 85 FPGA Board")
+		(date "2025-01-06")
 		(rev "V0.1")
 		(company "ODHIN Unicamp")
