File: ethernet.kicad_sch (KiCad schematic)
At the start: 0 parts

Commit message: Adicionando novos datasheets e comecando power
Parts:
- added C26, C27, C28, C29: 100n, symbol Device:C
- added C30, C31: 22p, symbol Device:C
- added J2: RJ45_JK0654219, Connector_RJ:RJ45_Pulse_JK0654219NL_Horizontal, symbol Connector:RJ45_JK0654219
- added R25: 12.1k, symbol Device:R
- added R3, R4: 1K, symbol Device:R
- added U7: KSZ9031RNXCA, Package_DFN_QFN:QFN-48-1EP_7x7mm_P0.5mm_EP5.15x5.15mm, symbol Interface_Ethernet:KSZ9031RNXCA
- added Y1: 25MHz, symbol Device:Crystal_GND3
Connections:
- new net: C30.1, U7.45 (XO), Y1.2
- new net: C31.1, U7.46 (XI), Y1.1
- new net: R25.2, U7.48 (ISET)
- new net: J2.16 (LED1+), R4.2
- new net: C27.2, J2.1 (MXCT3)
- new net: C28.2, J2.6 (MXCT2)
- new net: J2.14 (LED2+), R3.1
- new net: C29.2, J2.12 (MXCT1)
- new net: C26.2, J2.7 (MXCT4)
- new net ETH_LED1: R4.1
- new net ETH_LED2: R3.2
- new net GND: C26.1, C27.1, C28.1, C29.1, C30.2, C31.2, J2.13 (LED2-), J2.15 (LED1-), J2.SH, R25.1, U7.29 (VSS), U7.49 (PAD_GND), Y1.3
- new net MX1+: J2.11 (MX1+), U7.2 (TXRXP_A)
- new net MX1-: J2.10 (MX1-), U7.3 (TXRXM_A)
- new net MX2+: J2.4 (MX2+), U7.5 (TXRXP_B)
- new net MX2-: J2.5 (MX2-), U7.6 (TXRXM_B)
- new net MX3+: J2.3 (MX3+), U7.7 (TXRXP_C)
- new net MX3-: J2.2 (MX3-), U7.8 (TXRXM_C)
- new net MX4+: J2.8 (MX4+), U7.10 (TXRXP_D)
- new net MX4-: J2.9 (MX4-), U7.11 (TXRXM_D)
- no-connect marks 0 -> 1
Other:
- title: ECP5 85F Platonic Board -> PatchLogic 85 FPGA Board
