File: sdcard.kicad_sch (KiCad schematic)
At the start: 3 parts, among them J1 Micro_SD_Card

Commit message: Adicionando novos datasheets e comecando power
Other:
- title: ECP5 85F Platonic Board -> PatchLogic 85 FPGA Board
Changed lines of the file:
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@@
 	(paper "A4")
 	(title_block
-		(title "ECP5 85F Platonic Board")
+		(title "PatchLogic 85 FPGA Board")
 		(date "2025-01-05")
 		(rev "V0.1")
