File: clock.kicad_sch (KiCad schematic)
At the start: 0 parts

Commit message: Adicionando novos datasheets e comecando power
Other:
- title: ECP5 85F Platonic Board -> PatchLogic 85 FPGA Board
Changed lines of the file:
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@@
 	(paper "A4")
 	(title_block
-		(title "ECP5 85F Platonic Board")
+		(title "PatchLogic 85 FPGA Board")
 		(rev "V0.1")
 		(company "ODHIN Unicamp")

Commit message: Implementando power e ligando jtag e flash a fpga
Implementando circuito de power. Ligando JTAG e memoria FLASH quad SPI a
FPGA. Iniciando implementacão da DRAM e outros modulos
Parts:
- added C52: 1u, symbol Device:C
- added C53: C, symbol Device:C
- added FB6: 600R, symbol Device:FerriteBead
- added X2: 50MHz, Oscillator:Oscillator_SMD_EuroQuartz_XO32-4Pin_3.2x2.5mm, symbol Oscillator:XO32
Connections:
- new net: C52.1, C53.1, FB6.2, X2.4 (V+)
- new net +3V3: FB6.1
- new net FPGA_SYS_CLK: X2.3 (OUT)
- new net GND: C52.2, C53.2, X2.2 (GND)
- no-connect marks 0 -> 1
