File: dram.kicad_sch (KiCad schematic)
At the start: 0 parts

Commit message: Adicionando novos datasheets e comecando power
Other:
- title: ECP5 85F Platonic Board -> PatchLogic 85 FPGA Board
Changed lines of the file:
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@@
 	(paper "A4")
 	(title_block
-		(title "ECP5 85F Platonic Board")
+		(title "PatchLogic 85 FPGA Board")
 		(rev "V0.1")
 		(company "ODHIN Unicamp")

Commit message: Implementando power e ligando jtag e flash a fpga
Implementando circuito de power. Ligando JTAG e memoria FLASH quad SPI a
FPGA. Iniciando implementacão da DRAM e outros modulos
Parts:
- added U19: AS4C256M16D3, Package_BGA:BGA-96_9.0x13.0mm_Layout2x3x16_P0.8mm, symbol Memory_RAM:AS4C256M16D3
- added U20: TPS51200DRC, Package_SON:VSON-10-1EP_3x3mm_P0.5mm_EP1.65x2.4mm, symbol Regulator_Linear:TPS51200DRC
Connections:
- new net: U20.11 (GND), U20.4 (GND), U20.8 (GND)
- new net: U19.A1 (VDDQ), U19.A8 (VDDQ), U19.C1 (VDDQ), U19.C9 (VDDQ), U19.D2 (VDDQ), U19.E9 (VDDQ), U19.F1 (VDDQ), U19.H2 (VDDQ), U19.H9 (VDDQ)
- new net: U19.B2 (VDD), U19.D9 (VDD), U19.G7 (VDD), U19.K2 (VDD), U19.K8 (VDD), U19.N1 (VDD), U19.N9 (VDD), U19.R1 (VDD), U19.R9 (VDD)
- new net GND: U19.A9 (VSS), U19.B1 (VSSQ), U19.B3 (VSS), U19.B9 (VSSQ), U19.D1 (VSSQ), U19.D8 (VSSQ), U19.E1 (VSS), U19.E2 (VSSQ), U19.E8 (VSSQ), U19.F9 (VSSQ), U19.G1 (VSSQ), U19.G8 (VSS), U19.G9 (VSSQ), U19.J2 (VSS), U19.J8 (VSS), U19.M1 (VSS), U19.M9 (VSS), U19.P1 (VSS), U19.P9 (VSS), U19.T1 (VSS), U19.T9 (VSS)
